Commit message: kart description

File: src/kart_description/urdf/kart_urdf.urdf (robot description, URDF)
Before this commit: robot kart_urdf, 13 links, 12 joints
Links:
- link base_link: geometry collision mesh filename=package://kart_description/meshes/base_link.STL; visual mesh filename=package://kart_description/meshes/base_link.STL
- link battery_link: geometry collision mesh filename=package://kart_description/meshes/battery_link.STL; visual mesh filename=package://kart_description/meshes/battery_link.STL
- link lidar_link: geometry collision mesh filename=package://kart_description/meshes/lidar_link.STL; visual mesh filename=package://kart_description/meshes/lidar_link.STL
- link pivot_bl_link: geometry collision mesh filename=package://kart_description/meshes/pivot_bl_link.STL; visual mesh filename=package://kart_description/meshes/pivot_bl_link.STL
- link pivot_br_link: geometry collision mesh filename=package://kart_description/meshes/pivot_br_link.STL; visual mesh filename=package://kart_description/meshes/pivot_br_link.STL
- link pivot_fl_link: geometry collision mesh filename=package://kart_description/meshes/pivot_fl_link.STL; visual mesh filename=package://kart_description/meshes/pivot_fl_link.STL
- link pivot_fr_link: geometry collision mesh filename=package://kart_description/meshes/pivot_fr_link.STL; visual mesh filename=package://kart_description/meshes/pivot_fr_link.STL
- link plate_f_link: geometry collision mesh filename=package://kart_description/meshes/plate_f_link.STL; visual mesh filename=package://kart_description/meshes/plate_f_link.STL
- link plate_r_link: geometry collision mesh filename=package://kart_description/meshes/plate_r_link.STL; visual mesh filename=package://kart_description/meshes/plate_r_link.STL
- link wheel_bl_link: geometry collision mesh filename=package://kart_description/meshes/wheel_bl_link.STL; visual mesh filename=package://kart_description/meshes/wheel_bl_link.STL
- link wheel_br_link: geometry collision mesh filename=package://kart_description/meshes/wheel_br_link.STL; visual mesh filename=package://kart_description/meshes/wheel_br_link.STL
- link wheel_fl_link: geometry collision mesh filename=package://kart_description/meshes/wheel_fl_link.STL; visual mesh filename=package://kart_description/meshes/wheel_fl_link.STL
- link wheel_fr_link: geometry collision mesh filename=package://kart_description/meshes/wheel_fr_link.STL; visual mesh filename=package://kart_description/meshes/wheel_fr_link.STL

Commit message: corrected kart description, working on gazebo sim

File: src/kart_description/urdf/kart_urdf.urdf (robot description, URDF)
Before this commit: robot kart_description, 13 links, 12 joints
Links:
- added link dummy
Joints:
- added joint dummy_to_base_link=: type fixed, parent dummy, child base_link

Commit message: able to launch gazebo simulation. TODO: add plugins

File: src/kart_description/urdf/kart_urdf.urdf (robot description, URDF)
Before this commit: robot kart_description, 14 links, 13 joints
Links:
- link base_link: geometry collision mesh filename=file://$(find kart_description)/meshes/base_link.STL; visual mesh filename=file://$(find kart_description)/meshes/base_link.STL
- link battery_link: geometry collision mesh filename=file://$(find kart_description)/meshes/battery_link.STL; visual mesh filename=file://$(find kart_description)/meshes/battery_link.STL
- link lidar_link: geometry collision mesh filename=file://$(find kart_description)/meshes/lidar_link.STL; visual mesh filename=file://$(find kart_description)/meshes/lidar_link.STL
- link pivot_bl_link: geometry collision mesh filename=file://$(find kart_description)/meshes/pivot_bl_link.STL; visual mesh filename=file://$(find kart_description)/meshes/pivot_bl_link.STL
- link pivot_br_link: geometry collision mesh filename=file://$(find kart_description)/meshes/pivot_br_link.STL; visual mesh filename=file://$(find kart_description)/meshes/pivot_br_link.STL
- link pivot_fl_link: geometry collision mesh filename=file://$(find kart_description)/meshes/pivot_fl_link.STL; visual mesh filename=file://$(find kart_description)/meshes/pivot_fl_link.STL
- link pivot_fr_link: geometry collision mesh filename=file://$(find kart_description)/meshes/pivot_fr_link.STL; visual mesh filename=file://$(find kart_description)/meshes/pivot_fr_link.STL
- link plate_f_link: geometry collision mesh filename=file://$(find kart_description)/meshes/plate_f_link.STL; visual mesh filename=file://$(find kart_description)/meshes/plate_f_link.STL
- link plate_r_link: geometry collision mesh filename=file://$(find kart_description)/meshes/plate_r_link.STL; visual mesh filename=file://$(find kart_description)/meshes/plate_r_link.STL
- link wheel_bl_link: geometry collision mesh filename=file://$(find kart_description)/meshes/wheel_bl_link.STL; visual mesh filename=file://$(find kart_description)/meshes/wheel_bl_link.STL
- link wheel_br_link: geometry collision mesh filename=file://$(find kart_description)/meshes/wheel_br_link.STL; visual mesh filename=file://$(find kart_description)/meshes/wheel_br_link.STL
- link wheel_fl_link: geometry collision mesh filename=file://$(find kart_description)/meshes/wheel_fl_link.STL; visual mesh filename=file://$(find kart_description)/meshes/wheel_fl_link.STL
- link wheel_fr_link: geometry collision mesh filename=file://$(find kart_description)/meshes/wheel_fr_link.STL; visual mesh filename=file://$(find kart_description)/meshes/wheel_fr_link.STL
