Commit message: backup for urdf testing

File: src/kart_description/urdf/base.urdf (robot description, URDF)
Before this commit: robot castor_wheel, 3 links, 2 joints
Links:
- added link base_footprint
- link base_link: mass 1 -> 29.552; geometry collision mesh filename=file://$(find kart_description)/meshes/kart.STL; visual mesh filename=file://$(find kart_description)/meshes/kart.STL
Joints:
- added joint kart_joint: type fixed, parent base_footprint, child base_link, origin xyz=0 0 0.237 rpy=0.0 0.0 0.0, axis 0.0 0.0 1.0, limit effort=100 velocity=100
- joint fr_pivot_joint: origin xyz=0.0 0.0 0.0 rpy=0.0 0.0 0.0 -> xyz=0.2675 -0.14775 0 rpy=0.0 0.0 0.0

File: src/kart_description/urdf/castor_wheel.xacro (robot description, xacro)
@@ -28,8 +28,8 @@
         </xacro:segment>
     </xacro:macro>
-    <!-- Call the wheel macro -->
+    <!-- Call the wheel macro
     <link name="base_link"/>
     <xacro:castor_wheel parent="base_link" joint_prefix="fr_" link_prefix="fr_">
         <origin xyz="0.0 0.0 0.0" rpy="0.0 0.0 0.0"/>
-    </xacro:castor_wheel>
+    </xacro:castor_wheel>-->
 </robot>

File: src/kart_description/urdf/wheel_prev.urdf (robot description, URDF)
Before this commit: robot castor_wheel, 3 links, 2 joints
Links:
- link base_link: mass 1 -> None
- link fr_pivot_link: geometry collision box size=0.13339 0.1 0.16504; visual mesh filename=package://kart_description/meshes/pivot.STL
- link fr_wheel_link: geometry collision sphere radius=0.1; visual mesh filename=package://kart_description/meshes/wheel.STL
