Commit message: [R] refactor to xacros and properties to include materials.

File: src/kart_description/urdf/base_segment.xacro (robot description, xacro)
@@ -8,9 +8,10 @@
 	<xacro:property name="obj_props" value="${properties['objects']}"/>
 	<!-- Include Materials xacro file -->
-	<xacro:include filename="${package}/urdf/materials.urdf.xacro"/>
+	<!-- <xacro:include filename="${package}/urdf/materials.urdf.xacro"/>-->
+	<xacro:property name="materials" value="${properties['materials']}"/>
 	<!-- Geometry Collision/Visual Macro -->
 	<xacro:macro
 		name="geom"
-		params="mesh:=1 scale_factor:=^|1.0 reflect:=^ props:=^ model:=^|'base'">
+		params="mesh:=1 scale_factor:=^|1.0 reflect:=^|1.0 props:=^ model:=^|'base'">
 		<xacro:if value="${mesh == 0}">
 			<origin xyz = "${props['v_origin']['v_x']} ${props['v_origin']['v_y']} ${props['v_origin']['v_z']}" rpy= "${props['v_origin']['v_roll']} ${props['v_origin']['v_pitch']} ${props['v_origin']['v_yaw']}"/>
@@ -47,5 +48,5 @@
 		params="link_prefix:=^|''
 				joint_prefix:=^|''
-				reflect:=^!1
+				reflect:=^|1
 				scale_factor:=^|1.0
 				mesh:=1
@@ -56,4 +57,5 @@
 		<xacro:property name="props" value="${obj_props[model]}"/>
 		<xacro:property name="II" value="${props['inertia']}"/>
+		<xacro:property name="color" value="${materials[material]['color']}"/>
 		<!-- Joint Definition -->
 		<joint name="${joint_prefix}${model}_joint" type="${props['joint_type']}">
@@ -82,5 +84,7 @@
 			<visual>
 				<xacro:geom mesh="${mesh}" scale_factor="${scale_factor}" reflect="${reflect}" model="${model}"/>
-				<material name="${material}"/>
+				<material name="${material}">
+					<color rgba="${color['r']} ${color['g']} ${color['b']} ${color['a']}" />
+				</material>
 			</visual>
 			<!-- Collision -->

File: src/kart_description/urdf/castor_wheel.xacro (robot description, xacro)
@@ -2,9 +2,8 @@
 <robot name="castor_wheel"
     xmlns:xacro="http://ros.org/wiki/xacro">
-    <!-- xacro description of a castor wheel segment -->
-    <!-- A segment is composed of a joint and the attached link -->
+    <!-- Package Path -->
     <xacro:property name="package" value="$(find kart_description)"/>
     <!-- Include segment xacro -->
-    <xacro:include filename="${package}/urdf/base_segment.urdf.xacro"/>
+    <xacro:include filename="${package}/urdf/base_segment.xacro"/>
     <!-- CASTOR WHEEL MODEL -->
     <xacro:macro name="castor_wheel"
@@ -15,5 +14,5 @@
                         scale_factor:=^|1.0">
         <!-- PIVOT -->
-        <xacro:segment joint="pivot" link="pivot" parent="${parent}" model="pivot" material="Aluminum" mesh="1">
+        <xacro:segment joint="pivot" link="pivot" parent="${parent}" model="pivot" material="metal" mesh="1">
                 <!-- This origin comes from the file where the macro will be expanded -->
                 <xacro:insert_block name="origin"/>
@@ -22,5 +21,5 @@
         </xacro:segment>
         <!-- WHEEL -->
-        <xacro:segment joint="wheel" link="wheel" parent="${link_prefix}pivot_link" model="wheel" material="Rubber" mesh="1">
+        <xacro:segment joint="wheel" link="wheel" parent="${link_prefix}pivot_link" model="wheel" material="rubber" mesh="1">
                 <!--
                     This origin is fixed and belongs to the pivotal joint.
@@ -34,8 +33,9 @@
     </xacro:macro>
     <!-- Call the wheel macro -->
-    <link name="base_link"/>
+    <!--<link name="base_link"/>
     <xacro:castor_wheel parent="base_link"
                         joint_prefix="fr_" link_prefix="fr_">
         <origin xyz="0.0 0.0 0.0" rpy="0.0 0.0 0.0"/>
     </xacro:castor_wheel>
+    -->
 </robot>

Commit message: [R] refactored some properties and added common properties for inertial calculation. Useless at he moment.

File: src/kart_description/urdf/base_segment.xacro (robot description, xacro)
@@ -2,12 +2,12 @@
 <robot xmlns:xacro="http://ros.org/wiki/xacro">
 	<!-- Package Path -->
-	<xacro:property name="package" value="$(find kart_description)"/>
+	<xacro:property name="package" value="$(find kart_description)" />
 	<!-- Load the properties for the object to render -->
-	<xacro:property name="props_file" value="${package}/config/properties.yaml"/>
-	<xacro:property name="properties" value="${xacro.load_yaml(props_file)}"/>
-	<xacro:property name="obj_props" value="${properties['objects']}"/>
+	<xacro:property name="props_file" value="${package}/config/properties.yaml" />
+	<xacro:property name="properties" value="${xacro.load_yaml(props_file)}" />
+	<xacro:property name="obj_props" value="${properties['objects']}" />
 	<!-- Include Materials xacro file -->
 	<!-- <xacro:include filename="${package}/urdf/materials.urdf.xacro"/>-->
-	<xacro:property name="materials" value="${properties['materials']}"/>
+	<xacro:property name="materials" value="${properties['materials']}" />
 	<!-- Geometry Collision/Visual Macro -->
 	<xacro:macro
@@ -15,8 +15,10 @@
 		params="mesh:=1 scale_factor:=^|1.0 reflect:=^|1.0 props:=^ model:=^|'base'">
 		<xacro:if value="${mesh == 0}">
-			<origin xyz = "${props['v_origin']['v_x']} ${props['v_origin']['v_y']} ${props['v_origin']['v_z']}" rpy= "${props['v_origin']['v_roll']} ${props['v_origin']['v_pitch']} ${props['v_origin']['v_yaw']}"/>
+			<origin
+				xyz="${props['v_origin']['v_x']} ${props['v_origin']['v_y']} ${props['v_origin']['v_z']}"
+				rpy="${props['v_origin']['v_roll']} ${props['v_origin']['v_pitch']} ${props['v_origin']['v_yaw']}" />
 		</xacro:if>
 		<xacro:if value="${mesh == 1}">
-			<origin xyz = "0 0 0" rpy= "0 0 0"/>
+			<origin xyz="0 0 0" rpy="0 0 0" />
 		</xacro:if>
 		<geometry>
@@ -24,16 +26,26 @@
 			<xacro:if value="${mesh == 1}">
 				<!-- Load the mesh -->
-				<xacro:property name="mesh" value="${model}"/>
-				<mesh filename="package://${package.split('/')[-1]}/meshes/${mesh}.STL"/>
-				<!--scale="${scale_factor*0.001*reflect} ${scale_factor*0.001} ${scale_factor*0.001}"-->
+				<xacro:property name="mesh" value="${model}" />
+				<mesh filename="package://${package.split('/')[-1]}/meshes/${mesh}.STL" />
+				<!--scale="${scale_factor*0.001*reflect}
+				${scale_factor*0.001} ${scale_factor*0.001}"-->
 			</xacro:if>
 			<!-- Check which type of object is being loaded by its properties -->
 			<xacro:if value="${mesh == 0}">
 				<xacro:if value="${props['figure'] == 'cylinder'}">
-					<cylinder radius="${props['radius']*scale_factor}" length="${props['length']*scale_factor}"/>
+					<cylinder radius="${props['radius']*scale_factor}"
+						length="${props['length']*scale_factor}" />
 				</xacro:if>
 				<xacro:if value="${props['figure'] == 'box'}">
-					<box size="${props['width']} ${props['length']} ${props['height']}"/>
-					<origin xyz="0 0 ${props['height']/2.0}" rpy="0 0 0"/>
+					<box size="${props['width']} ${props['length']} ${props['height']}" />
+					<origin xyz="0 0 ${props['height']/2.0}" rpy="0 0 0" />
+				</xacro:if>
+				<xacro:if value="${props['figure'] == 'sphere'}">
+					<sphere radius="${props['radius']*scale_factor}" />
+				</xacro:if>
+				<xacro:if value="${props['figure'] == 'mesh'}">
+					<mesh filename="package://${package.split('/')[-1]}/meshes/${model}.STL" />
+					<!--scale="${scale_factor*0.001*reflect}
+					${scale_factor*0.001} ${scale_factor*0.001}"-->
 				</xacro:if>
 			</xacro:if>
@@ -55,33 +67,37 @@
 				model:=^|'base'
 				joint link parent">
-		<xacro:property name="props" value="${obj_props[model]}"/>
-		<xacro:property name="II" value="${props['inertia']}"/>
-		<xacro:property name="color" value="${materials[material]['color']}"/>
+		<xacro:property name="props" value="${obj_props[model]}" />
+		<xacro:property name="II" value="${props['inertia']}" />
+		<xacro:property name="color" value="${materials[material]['color']}" />
 		<!-- Joint Definition -->
 		<joint name="${joint_prefix}${model}_joint" type="${props['joint_type']}">
-			<parent link="${parent}"/>
-			<child link="${link_prefix}${model}_link"/>
-			<xacro:insert_block name="origin"/>
-			<xacro:insert_block name="axis"/>
+			<parent link="${parent}" />
+			<child link="${link_prefix}${model}_link" />
+			<xacro:insert_block name="origin" />
+			<xacro:insert_block name="axis" />
 			<!-- add bounds for the joint if present in the config file -->
 			<xacro:if value="${'bounds' in props.keys()}">
-				<limit lower="${props['bounds']['lower']*pi/180}" upper="${props['bounds']['upper']*pi/180}" effort="${props['effort']}" velocity="${props['velocity']}"/>
+				<limit lower="${props['bounds']['lower']*pi/180}"
+					upper="${props['bounds']['upper']*pi/180}" effort="${props['effort']}"
+					velocity="${props['velocity']}" />
 			</xacro:if>
 			<!-- If not, just add limits and dynamics factors -->
 			<xacro:if value="${'bounds' not in props.keys()}">
-				<limit effort="${props['effort']}" velocity="${props['velocity']}"/>
+				<limit effort="${props['effort']}" velocity="${props['velocity']}" />
 			</xacro:if>
-			<dynamics damping="${props['damping']}" friction="${props['friction']}"/>
+			<dynamics damping="${props['damping']}" friction="${props['friction']}" />
 		</joint>
 		<!-- Link Definition -->
 		<link name="${link_prefix}${model}_link">
-			<intertial>
-				<mass value="${props['mass']}"/>
-				<inertia ixx="${II['ixx']}" iyy="${II['iyy']}" izz="${II['izz']}" ixy="${II['ixy']}" iyz="${II['iyz']}" ixz="${II['ixz']}"/>
-				<origin xyz="${II['xyz']}" rpy="${II['rpy']}"/>
-			</intertial>
+			<inertial>
+				<mass value="${props['mass']}" />
+				<inertia ixx="${II['ixx']}" iyy="${II['iyy']}" izz="${II['izz']}" ixy="${II['ixy']}"
+					iyz="${II['iyz']}" ixz="${II['ixz']}" />
+				<origin xyz="${II['xyz']}" rpy="${II['rpy']}" />
+			</inertial>
 			<!-- Geometry -->
 			<visual>
-				<xacro:geom mesh="${mesh}" scale_factor="${scale_factor}" reflect="${reflect}" model="${model}"/>
+				<xacro:geom mesh="${mesh}" scale_factor="${scale_factor}" reflect="${reflect}"
+					model="${model}" />
 				<material name="${material}">
 					<color rgba="${color['r']} ${color['g']} ${color['b']} ${color['a']}" />
@@ -90,5 +106,6 @@
 			<!-- Collision -->
 			<collision>
-				<xacro:geom mesh="0" scale_factor="${scale_factor}" reflect="${reflect}" model="${model}"/>
+				<xacro:geom mesh="0" scale_factor="${scale_factor}" reflect="${reflect}"
+					model="${model}" />
 			</collision>
 		</link>

File: src/kart_description/urdf/castor_wheel.xacro (robot description, xacro)
@@ -7,35 +7,29 @@
     <xacro:include filename="${package}/urdf/base_segment.xacro"/>
     <!-- CASTOR WHEEL MODEL -->
-    <xacro:macro name="castor_wheel"
-                params="parent
-                        link_prefix:=^|''
-                        joint_prefix:=^|''
-                        *origin
-                        scale_factor:=^|1.0">
+    <xacro:macro name="castor_wheel" params="parent link_prefix:=^|'' joint_prefix:=^|''
+                        *origin scale_factor:=^|1.0">
         <!-- PIVOT -->
         <xacro:segment joint="pivot" link="pivot" parent="${parent}" model="pivot" material="metal" mesh="1">
-                <!-- This origin comes from the file where the macro will be expanded -->
-                <xacro:insert_block name="origin"/>
-                <!-- The rotation happens on the Z-axis -->
-                <axis xyz="0.0 0.0 1.0"/>
+            <!-- This origin comes from the file where the macro will be expanded -->
+            <xacro:insert_block name="origin"/>
+            <!-- The rotation happens on the Z-axis -->
+            <axis xyz="0.0 0.0 1.0"/>
         </xacro:segment>
         <!-- WHEEL -->
         <xacro:segment joint="wheel" link="wheel" parent="${link_prefix}pivot_link" model="wheel" material="rubber" mesh="1">
-                <!--
+            <!--
                     This origin is fixed and belongs to the pivotal joint.
                     To rotate the wheel around its own axis, we need to rotate
                     the mesh around the X-axis
                 -->
-                <origin xyz="-0.059 0 -0.14065" rpy="${pi/2} 0.0 0.0"/>
-                <!-- The rotation happens on the Z-axis -->
-                <axis xyz="0.0 0.0 1.0"/>
+            <origin xyz="-0.059 0 -0.14065" rpy="${pi/2} 0.0 0.0"/>
+            <!-- The rotation happens on the Z-axis -->
+            <axis xyz="0.0 0.0 1.0"/>
         </xacro:segment>
     </xacro:macro>
     <!-- Call the wheel macro -->
-    <!--<link name="base_link"/>
-    <xacro:castor_wheel parent="base_link"
-                        joint_prefix="fr_" link_prefix="fr_">
+    <link name="base_link"/>
+    <xacro:castor_wheel parent="base_link" joint_prefix="fr_" link_prefix="fr_">
         <origin xyz="0.0 0.0 0.0" rpy="0.0 0.0 0.0"/>
     </xacro:castor_wheel>
-    -->
 </robot>

Commit message: working on xacro files

File: src/kart_description/urdf/base_segment.xacro (robot description, xacro)
@@ -66,5 +66,5 @@
 				*origin *axis
 				model:=^|'base'
-				joint link parent">
+				parent">
 		<xacro:property name="props" value="${obj_props[model]}" />
 		<xacro:property name="II" value="${props['inertia']}" />
@@ -76,15 +76,18 @@
 			<xacro:insert_block name="origin" />
 			<xacro:insert_block name="axis" />
-			<!-- add bounds for the joint if present in the config file -->
-			<xacro:if value="${'bounds' in props.keys()}">
-				<limit lower="${props['bounds']['lower']*pi/180}"
-					upper="${props['bounds']['upper']*pi/180}" effort="${props['effort']}"
-					velocity="${props['velocity']}" />
+			<!-- If the joint isn't a fixed one add range and dynamic properties -->
+			<xacro:if value="${props['joint_type'] != 'fixed'}">
+				<!-- add bounds for the joint if present in the config file -->
+				<xacro:if value="${'bounds' in props.keys()}">
+					<limit lower="${props['bounds']['lower']*pi/180}"
+						upper="${props['bounds']['upper']*pi/180}" effort="${props['effort']}"
+						velocity="${props['velocity']}" />
+				</xacro:if>
+				<!-- If not, just add limits and dynamics factors -->
+				<xacro:if value="${'bounds' not in props.keys()}">
+					<limit effort="${props['effort']}" velocity="${props['velocity']}" />
+				</xacro:if>
+				<dynamics damping="${props['damping']}" friction="${props['friction']}" />
 			</xacro:if>
-			<!-- If not, just add limits and dynamics factors -->
-			<xacro:if value="${'bounds' not in props.keys()}">
-				<limit effort="${props['effort']}" velocity="${props['velocity']}" />
-			</xacro:if>
-			<dynamics damping="${props['damping']}" friction="${props['friction']}" />
 		</joint>
 		<!-- Link Definition -->

File: src/kart_description/urdf/castor_wheel.xacro (robot description, xacro)
@@ -10,5 +10,5 @@
                         *origin scale_factor:=^|1.0">
         <!-- PIVOT -->
-        <xacro:segment joint="pivot" link="pivot" parent="${parent}" model="pivot" material="metal" mesh="1">
+        <xacro:segment parent="${parent}" model="pivot" material="metal" mesh="1">
             <!-- This origin comes from the file where the macro will be expanded -->
             <xacro:insert_block name="origin"/>
@@ -17,5 +17,5 @@
         </xacro:segment>
         <!-- WHEEL -->
-        <xacro:segment joint="wheel" link="wheel" parent="${link_prefix}pivot_link" model="wheel" material="rubber" mesh="1">
+        <xacro:segment parent="${link_prefix}pivot_link" model="wheel" material="rubber" mesh="1">
             <!--
                     This origin is fixed and belongs to the pivotal joint.

File: src/kart_description/urdf/kart_base.xacro (robot description, xacro)
@@ -9,5 +9,5 @@
     <xacro:macro name="kart_base" params="parent link_prefix:=^|'' joint_prefix:=^|'' *origin scale_factor:=^|1.0">
         <!-- BASE -->
-        <xacro:segment joint="base_joint" link="base_link" parent="${parent}" model="kart" material="metal" mesh="1">
+        <xacro:segment parent="${parent}" model="kart" material="metal" mesh="1">
             <!-- This origin comes from the file where the macro will be expanded -->
             <xacro:insert_block name="origin"/>
@@ -16,13 +16,13 @@
         </xacro:segment>
     </xacro:macro>
-    <!-- Call the base macro -->
+    <!-- Call the base macro
     <link name="base_footprint"/>
     <xacro:kart_base parent="base_footprint" joint_prefix="" link_prefix="">
-        <origin xyz="0 0 0.3" rpy="0.0 0.0 0.0"/>
-    </xacro:kart_base>
-    <!-- Include the wheels -->
+        <origin xyz="0 0 0" rpy="0.0 0.0 0.0"/>
+    </xacro:kart_base>-->
+    <!-- Include the wheels
     <xacro:include filename="${package}/urdf/castor_wheel.xacro"/>
     <xacro:castor_wheel parent="base_link" joint_prefix="fr_" link_prefix="fr_">
         <origin xyz="0.2675 -0.14775 0" rpy="0.0 0.0 0.0"/>
-    </xacro:castor_wheel>
+    </xacro:castor_wheel> -->
 </robot>

File: src/kart_description/urdf/wheel_prev.urdf (robot description, URDF)
Before this commit: robot castor_wheel, 3 links, 2 joints
Links:
- link fr_pivot_link: mass 4.9241947653983 -> 1.2
- link fr_wheel_link: mass 1.9175 -> 1.22
