Commit message: testing gazebo integration

File: src/kart_description/urdf/kart.urdf (robot description, URDF)
Before this commit: robot kart, 12 links, 11 joints
Links:
- link fl_pivot_link: mass 4.9241947653983 -> 1.2
- link fl_wheel_link: mass 1.9175 -> 1.22
- link fr_pivot_link: mass 4.9241947653983 -> 1.2
- link fr_wheel_link: mass 1.9175 -> 1.22
- link rl_pivot_link: mass 4.9241947653983 -> 1.2
- link rl_wheel_link: mass 1.9175 -> 1.22
- link rr_pivot_link: mass 4.9241947653983 -> 1.2
- link rr_wheel_link: mass 1.9175 -> 1.22
Joints:
- joint base_joint: origin xyz=0 0 0 rpy=0.0 0.0 0.0 -> xyz=0 0 0.242 rpy=0.0 0.0 0.0

File: src/kart_description/urdf/mobile_base_gazebo.xacro (robot description, xacro)
@@ -1,3 +1,31 @@
 <?xml version="1.0" encoding="UTF-8"?>
 <robot xmlns:xacro="http://www.ros.org/wiki/xacro">
+    <!-- Edit Friction in simulation -->
+    <gazebo reference="base_link">
+        <mu1>0.000002</mu1>
+        <mu2>0.000002</mu2>
+    </gazebo>
+    <!-- Diff Drive Plugin -->
+    <gazebo>
+        <plugin
+            filename="gz-sim-diff-drive-system"
+            name="gz::sim::systems::DiffDrive">
+            <left_joint>fl_wheel_joint</left_joint>
+            <right_joint>fr_wheel_joint</right_joint>
+            <frame_id>odom</frame_id>
+            <child_frame_id>base_footprint</child_frame_id>
+            <wheel_separation>0.29549</wheel_separation>
+            <wheel_radius>0.1</wheel_radius>
+            <max_acceleration>0.3</max_acceleration>
+        </plugin>
+    </gazebo>
+    <!-- Publish Joint State Info -->
+    <gazebo>
+        <plugin
+            filename="gz-sim-joint-state-publisher-system"
+            name="gz::sim::systems::JointStatePublisher">
+            <update_rate>50</update_rate>
+            <publish_tf>true</publish_tf>
+        </plugin>
+    </gazebo>
 </robot>
